Commit message: reorganized: renamed and organized description package

File: mh180_description/urdf/mh180_120.urdf.xacro (robot description, xacro)
@@ -1,5 +1,5 @@
 <?xml version="1.0" ?>
 <robot name="motoman_mh_180_120" xmlns:xacro="http://ros.org/wiki/xacro">
-  <xacro:include filename="$(find yaskawa_motoman_description)/urdf/mh180_120_macro.urdf.xacro"/>
+  <xacro:include filename="$(find mh180_description)/urdf/mh180_120_macro.urdf.xacro"/>
   <xacro:motoman_mh180_120 prefix=""/>
 </robot>

File: mh180_description/urdf/mh180_120_macro.urdf.xacro (robot description, xacro)
@@ -7,5 +7,5 @@
         <origin xyz="0 0 0" rpy="0 0 0"/>
         <geometry>
-          <mesh filename="package://yaskawa_motoman_description/meshes/mh180/visual/base_link.stl"/>
+          <mesh filename="package://mh180_description/meshes/mh180/visual/base_link.stl"/>
         </geometry>
         <material name="blue">
@@ -16,5 +16,5 @@
       	<origin xyz="0 0 0" rpy="0 0 0"/>
         <geometry>
-          <mesh filename="package://yaskawa_motoman_description/meshes/mh180/collision/base_link.stl"/>
+          <mesh filename="package://mh180_description/meshes/mh180/collision/base_link.stl"/>
           <!--box size="0.9 0.5 0.32"/-->
         </geometry>
@@ -28,5 +28,5 @@
         <origin xyz="0 0 0" rpy="0 0 0"/>
         <geometry>
-          <mesh filename="package://yaskawa_motoman_description/meshes/mh180/visual/link_s.stl"/>
+          <mesh filename="package://mh180_description/meshes/mh180/visual/link_s.stl"/>
         </geometry>
         <material name="blue"/>
@@ -35,5 +35,5 @@
         <origin xyz="0 0 0" rpy="0 0 0"/>
         <geometry>
-          <mesh filename="package://yaskawa_motoman_description/meshes/mh180/collision/link_s.stl"/>
+          <mesh filename="package://mh180_description/meshes/mh180/collision/link_s.stl"/>
         </geometry>
         <material name="yellow"/>
@@ -44,5 +44,5 @@
         <origin xyz="0 0 0" rpy="0 0 0"/>
         <geometry>
-          <mesh filename="package://yaskawa_motoman_description/meshes/mh180/visual/link_l.stl"/>
+          <mesh filename="package://mh180_description/meshes/mh180/visual/link_l.stl"/>
         </geometry>
         <material name="blue"/>
@@ -51,5 +51,5 @@
         <origin xyz="0 0 0" rpy="0 0 0"/>
         <geometry>
-          <mesh filename="package://yaskawa_motoman_description/meshes/mh180/collision/link_l.stl"/>
+          <mesh filename="package://mh180_description/meshes/mh180/collision/link_l.stl"/>
         </geometry>
         <material name="yellow"/>
@@ -60,5 +60,5 @@
         <origin xyz="0 0 0" rpy="0 0 0"/>
         <geometry>
-          <mesh filename="package://yaskawa_motoman_description/meshes/mh180_120/visual/link_u.stl"/>
+          <mesh filename="package://mh180_description/meshes/mh180/visual/link_u.stl"/>
         </geometry>
         <material name="blue"/>
@@ -67,5 +67,5 @@
         <origin xyz="0 0 0" rpy="0 0 0"/>
         <geometry>
-          <mesh filename="package://yaskawa_motoman_description/meshes/mh180_120/collision/link_u.stl"/>
+          <mesh filename="package://mh180_description/meshes/mh180/collision/link_u.stl"/>
         </geometry>
         <material name="yellow"/>
@@ -76,5 +76,5 @@
         <origin xyz="0 0 0" rpy="0 0 0"/>
         <geometry>
-          <mesh filename="package://yaskawa_motoman_description/meshes/mh180_120/visual/link_r.stl"/>
+          <mesh filename="package://mh180_description/meshes/mh180/visual/link_r.stl"/>
         </geometry>
         <material name="blue"/>
@@ -83,5 +83,5 @@
         <origin xyz="0 0 0" rpy="0 0 0"/>
         <geometry>
-          <mesh filename="package://yaskawa_motoman_description/meshes/mh180_120/collision/link_r.stl"/>
+          <mesh filename="package://mh180_description/meshes/mh180/collision/link_r.stl"/>
         </geometry>
         <material name="yellow"/>
@@ -92,5 +92,5 @@
         <origin xyz="0 0 0" rpy="0 0 0"/>
         <geometry>
-          <mesh filename="package://yaskawa_motoman_description/meshes/mh180/visual/link_b.stl"/>
+          <mesh filename="package://mh180_description/meshes/mh180/visual/link_b.stl"/>
         </geometry>
         <material name="blue"/>
@@ -99,5 +99,5 @@
         <origin xyz="0 0 0" rpy="0 0 0"/>
         <geometry>
-          <mesh filename="package://yaskawa_motoman_description/meshes/mh180/collision/link_b.stl"/>
+          <mesh filename="package://mh180_description/meshes/mh180/collision/link_b.stl"/>
         </geometry>
         <material name="yellow"/>
@@ -108,5 +108,5 @@
         <origin xyz="0 0 0" rpy="0 0 0"/>
         <geometry>
-          <mesh filename="package://yaskawa_motoman_description/meshes/mh180/visual/link_t.stl"/>
+          <mesh filename="package://mh180_description/meshes/mh180/visual/link_t.stl"/>
         </geometry>
         <material name="black">
@@ -117,5 +117,5 @@
         <origin xyz="0 0 0" rpy="0 0 0"/>
         <geometry>
-          <mesh filename="package://yaskawa_motoman_description/meshes/mh180/collision/link_t.stl"/>
+          <mesh filename="package://mh180_description/meshes/mh180/collision/link_t.stl"/>
         </geometry>
         <material name="black"/>
